File: Hardware/Panel/dso138_panel/dso138_panel.kicad_sch (KiCad schematic)
At the start: 27 parts

Commit message: TO-220 regulator; panel
Parts:
- GRAF1, GRAF2: symbol ao_symbols:Graphic -> AO_symbols:Graphic
- GRAF3: footprint ao_tht:CC0_logo -> AO_tht:CC0_logo; symbol ao_symbols:Graphic -> AO_symbols:Graphic
- H23, H24: footprint Kosmo_panel:Kosmo_Panel_Dual_Slotted_Mounting_Holes -> Kosmo_panel_NPTH:Kosmo_Panel_Dual_Slotted_Mounting_Holes

Commit message: gerbers
Parts:
- H1, H11, H15, H16, H6: footprint Kosmo_panel_NPTH:Kosmo_Tact_Button_13mm_square_Hole -> Kosmo_panel:Kosmo_Tact_Button_13mm_square_Hole
- H10, H5: footprint Kosmo_panel_NPTH:Kosmo_Switch_Hole -> Kosmo_panel:Kosmo_Switch_Hole
- H12, H2, H7: footprint Kosmo_panel_NPTH:Kosmo_DP3T_Slide_Switch_Hole -> Kosmo_panel:Kosmo_DP3T_Slide_Switch_Hole
- H13, H17, H3, H8: footprint Kosmo_panel_NPTH:Kosmo_Panel_Mounting_Hole -> Kosmo_panel:Kosmo_Panel_Mounting_Hole
- H14, H9: footprint Kosmo_panel_NPTH:Kosmo_Jack_Hole -> Kosmo_panel:Kosmo_Jack_Hole
- H22: footprint Kosmo_panel_NPTH:Kosmo_LED_Hole -> Kosmo_panel:Kosmo_LED_Hole
- H23, H24: footprint Kosmo_panel_NPTH:Kosmo_Panel_Dual_Slotted_Mounting_Holes -> Kosmo_panel:Kosmo_Panel_Dual_Slotted_Mounting_Holes
- H4: footprint Kosmo_panel_NPTH:Kosmo_Push_Button_Daier_Hole -> Kosmo_panel:Kosmo_Push_Button_Daier_Hole
Changed lines of the file:
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@@
       (effects (font (size 1.27 1.27)) (justify left))
     )
-    (property "Footprint" "Kosmo_panel_NPTH:Kosmo_LED_Hole" (at 256.921 64.897 0)
+    (property "Footprint" "Kosmo_panel:Kosmo_LED_Hole" (at 256.921 64.897 0)
       (effects (font (size 1.27 1.27)) hide)
     )
@@
       (effects (font (size 1.27 1.27)) (justify left))
     )
-    (property "Footprint" "Kosmo_panel_NPTH:Kosmo_Tact_Button_13mm_square_Hole" (at 111.76 55.88 0)
+    (property "Footprint" "Kosmo_panel:Kosmo_Tact_Button_13mm_square_Hole" (at 111.76 55.88 0)
       (effects (font (size 1.27 1.27)) hide)
     )
@@
       (effects (font (size 1.27 1.27)) (justify left))
     )
-    (property "Footprint" "Kosmo_panel_NPTH:Kosmo_DP3T_Slide_Switch_Hole" (at 111.76 68.58 0)
+    (property "Footprint" "Kosmo_panel:Kosmo_DP3T_Slide_Switch_Hole" (at 111.76 68.58 0)
       (effects (font (size 1.27 1.27)) hide)
     )
@@
       (effects (font (size 1.27 1.27)) (justify left))
     )
-    (property "Footprint" "Kosmo_panel_NPTH:Kosmo_Panel_Dual_Slotted_Mounting_Holes" (at 127 124.46 0)
+    (property "Footprint" "Kosmo_panel:Kosmo_Panel_Dual_Slotted_Mounting_Holes" (at 127 124.46 0)
       (effects (font (size 1.27 1.27)) hide)
     )
@@
       (effects (font (size 1.27 1.27)) (justify left))
     )
-    (property "Footprint" "Kosmo_panel_NPTH:Kosmo_Jack_Hole" (at 111.76 105.41 0)
+    (property "Footprint" "Kosmo_panel:Kosmo_Jack_Hole" (at 111.76 105.41 0)
       (effects (font (size 1.27 1.27)) hide)
     )
@@
       (effects (font (size 1.27 1.27)) (justify left))
     )
-    (property "Footprint" "Kosmo_panel_NPTH:Kosmo_Push_Button_Daier_Hole" (at 58.42 104.14 0)
+    (property "Footprint" "Kosmo_panel:Kosmo_Push_Button_Daier_Hole" (at 58.42 104.14 0)
       (effects (font (size 1.27 1.27)) hide)
     )
@@
       (effects (font (size 1.27 1.27)) (justify left))
     )
-    (property "Footprint" "Kosmo_panel_NPTH:Kosmo_Panel_Mounting_Hole" (at 138.43 85.09 0)
+    (property "Footprint" "Kosmo_panel:Kosmo_Panel_Mounting_Hole" (at 138.43 85.09 0)
       (effects (font (size 1.27 1.27)) hide)
     )
@@
       (effects (font (size 1.27 1.27)) (justify left))
     )
-    (property "Footprint" "Kosmo_panel_NPTH:Kosmo_Switch_Hole" (at 85.725 120.396 0)
+    (property "Footprint" "Kosmo_panel:Kosmo_Switch_Hole" (at 85.725 120.396 0)
       (effects (font (size 1.27 1.27)) hide)
     )
@@
       (effects (font (size 1.27 1.27)) (justify left))
     )
-    (property "Footprint" "Kosmo_panel_NPTH:Kosmo_DP3T_Slide_Switch_Hole" (at 58.42 68.58 0)
+    (property "Footprint" "Kosmo_panel:Kosmo_DP3T_Slide_Switch_Hole" (at 58.42 68.58 0)
       (effects (font (size 1.27 1.27)) hide)
     )
@@
       (effects (font (size 1.27 1.27)) (justify left))
     )
-    (property "Footprint" "Kosmo_panel_NPTH:Kosmo_Tact_Button_13mm_square_Hole" (at 138.43 55.88 0)
+    (property "Footprint" "Kosmo_panel:Kosmo_Tact_Button_13mm_square_Hole" (at 138.43 55.88 0)
       (effects (font (size 1.27 1.27)) hide)
     )
@@
       (effects (font (size 1.27 1.27)) (justify left))
     )
-    (property "Footprint" "Kosmo_panel_NPTH:Kosmo_Panel_Mounting_Hole" (at 85.09 85.09 0)
+    (property "Footprint" "Kosmo_panel:Kosmo_Panel_Mounting_Hole" (at 85.09 85.09 0)
       (effects (font (size 1.27 1.27)) hide)
     )
@@
       (effects (font (size 1.27 1.27)) (justify left))
     )
-    (property "Footprint" "Kosmo_panel_NPTH:Kosmo_Switch_Hole" (at 59.055 120.396 0)
+    (property "Footprint" "Kosmo_panel:Kosmo_Switch_Hole" (at 59.055 120.396 0)
       (effects (font (size 1.27 1.27)) hide)
     )
@@
       (effects (font (size 1.27 1.27)) (justify left))
     )
-    (property "Footprint" "Kosmo_panel_NPTH:Kosmo_Jack_Hole" (at 85.09 105.41 0)
+    (property "Footprint" "Kosmo_panel:Kosmo_Jack_Hole" (at 85.09 105.41 0)
       (effects (font (size 1.27 1.27)) hide)
     )
@@
       (effects (font (size 1.27 1.27)) (justify left))
     )
-    (property "Footprint" "Kosmo_panel_NPTH:Kosmo_Tact_Button_13mm_square_Hole" (at 58.42 55.88 0)
+    (property "Footprint" "Kosmo_panel:Kosmo_Tact_Button_13mm_square_Hole" (at 58.42 55.88 0)
       (effects (font (size 1.27 1.27)) hide)
     )
@@
       (effects (font (size 1.27 1.27)) (justify left))
     )
-    (property "Footprint" "Kosmo_panel_NPTH:Kosmo_Tact_Button_13mm_square_Hole" (at 138.43 68.58 0)
+    (property "Footprint" "Kosmo_panel:Kosmo_Tact_Button_13mm_square_Hole" (at 138.43 68.58 0)
       (effects (font (size 1.27 1.27)) hide)
     )
@@
       (effects (font (size 1.27 1.27)) (justify left))
     )
-    (property "Footprint" "Kosmo_panel_NPTH:Kosmo_Panel_Mounting_Hole" (at 111.76 85.09 0)
+    (property "Footprint" "Kosmo_panel:Kosmo_Panel_Mounting_Hole" (at 111.76 85.09 0)
       (effects (font (size 1.27 1.27)) hide)
     )
@@
       (effects (font (size 1.27 1.27)) (justify left))
     )
-    (property "Footprint" "Kosmo_panel_NPTH:Kosmo_Tact_Button_13mm_square_Hole" (at 85.09 55.88 0)
+    (property "Footprint" "Kosmo_panel:Kosmo_Tact_Button_13mm_square_Hole" (at 85.09 55.88 0)
       (effects (font (size 1.27 1.27)) hide)
     )
@@
       (effects (font (size 1.27 1.27)) (justify left))
     )
-    (property "Footprint" "Kosmo_panel_NPTH:Kosmo_DP3T_Slide_Switch_Hole" (at 85.09 68.58 0)
+    (property "Footprint" "Kosmo_panel:Kosmo_DP3T_Slide_Switch_Hole" (at 85.09 68.58 0)
       (effects (font (size 1.27 1.27)) hide)
     )
@@
       (effects (font (size 1.27 1.27)) (justify left))
     )
-    (property "Footprint" "Kosmo_panel_NPTH:Kosmo_Panel_Dual_Slotted_Mounting_Holes" (at 152.4 124.46 0)
+    (property "Footprint" "Kosmo_panel:Kosmo_Panel_Dual_Slotted_Mounting_Holes" (at 152.4 124.46 0)
       (effects (font (size 1.27 1.27)) hide)
     )
@@
       (effects (font (size 1.27 1.27)) (justify left))
     )
-    (property "Footprint" "Kosmo_panel_NPTH:Kosmo_Panel_Mounting_Hole" (at 58.42 85.09 0)
-      (effects (font (size 1.27 1.27)) hide)
-    )
+    (property "Footprint" "Kosmo_panel:Kosmo_Panel_Mounting_Hole" (at 58.42 85.09 0)
+      (effects (font (size 1.27 1.27)) hide)
+    )
